Commit message: Added teleop template and controllers

File: pharmacy_robot/urdf/pharmacy_gripper.xacro (robot description, xacro)
@@ -494,4 +494,15 @@
 		<dynamics damping="5" friction="3" />
 	</joint>
+	<!-- Add transmission for robot_base joint -->
+  <transmission name="robot_base_trans">
+    <type>transmission_interface/SimpleTransmission</type>
+    <joint name="robot_base">
+      <hardwareInterface>PositionJointInterface</hardwareInterface>
+    </joint>
+    <actuator name="robot_base_motor">
+      <hardwareInterface>PositionJointInterface</hardwareInterface>
+      <mechanicalReduction>1</mechanicalReduction>
+    </actuator>
+  </transmission>
 	<joint name="vertical_rail" type="revolute">
 		<origin
@@ -511,4 +522,15 @@
 		<dynamics damping="5" friction="3" />
   	</joint>
+	<!-- Add transmission for vertical_rail joint -->
+  <transmission name="vertical_rail_trans">
+    <type>transmission_interface/SimpleTransmission</type>
+    <joint name="vertical_rail">
+      <hardwareInterface>PositionJointInterface</hardwareInterface>
+    </joint>
+    <actuator name="revolute_base_motor">
+      <hardwareInterface>PositionJointInterface</hardwareInterface>
+      <mechanicalReduction>1</mechanicalReduction>
+    </actuator>
+  </transmission>
 	<joint
 		name="prismatic_base"
@@ -530,4 +552,15 @@
 		<dynamics damping="5" friction="3" />
 	</joint>
+	<!-- Add transmission for prismatic_base joint -->
+  <transmission name="prismatic_base_trans">
+    <type>transmission_interface/SimpleTransmission</type>
+    <joint name="prismatic_base">
+      <hardwareInterface>PositionJointInterface</hardwareInterface>
+    </joint>
+    <actuator name="prismatic_base_motor">
+      <hardwareInterface>PositionJointInterface</hardwareInterface>
+      <mechanicalReduction>1</mechanicalReduction>
+    </actuator>
+  </transmission>
 	<joint
 		name="prismatic_arm"
@@ -549,4 +582,15 @@
 		<dynamics damping="5" friction="3" />
 	</joint>
+	<!-- Add transmission for prismatic_base joint -->
+  <transmission name="prismatic_arm_trans">
+    <type>transmission_interface/SimpleTransmission</type>
+    <joint name="prismatic_arm">
+      <hardwareInterface>PositionJointInterface</hardwareInterface>
+    </joint>
+    <actuator name="prismatic_arm_motor">
+      <hardwareInterface>PositionJointInterface</hardwareInterface>
+      <mechanicalReduction>1</mechanicalReduction>
+    </actuator>
+  </transmission>
 	<joint
 		name="gripper_base_"
@@ -568,4 +612,15 @@
 		<dynamics damping="5" friction="3" />
 	</joint>
+	<!-- Add transmission for prismatic_base joint -->
+  <transmission name="gripper_base_trans">
+    <type>transmission_interface/SimpleTransmission</type>
+    <joint name="gripper_base">
+      <hardwareInterface>PositionJointInterface</hardwareInterface>
+    </joint>
+    <actuator name="gripper_base_motor">
+      <hardwareInterface>PositionJointInterface</hardwareInterface>
+      <mechanicalReduction>1</mechanicalReduction>
+    </actuator>
+  </transmission>
 	<joint
 		name="camera"
@@ -593,4 +648,15 @@
         <limit lower="0.0" upper="0.8" velocity="0.5" effort="50" />
     </joint>
+	<!-- Add transmission for robotiq_85_left_knuckle_joint joint -->
+  <transmission name="robotiq_85_left_knuckle_joint_trans">
+    <type>transmission_interface/SimpleTransmission</type>
+    <joint name="robotiq_85_left_knuckle_joint">
+      <hardwareInterface>PositionJointInterface</hardwareInterface>
+    </joint>
+    <actuator name="robotiq_85_left_knuckle_joint_motor">
+      <hardwareInterface>PositionJointInterface</hardwareInterface>
+      <mechanicalReduction>1</mechanicalReduction>
+    </actuator>
+  </transmission>
     <joint name="robotiq_85_right_knuckle_joint" type="revolute">
         <parent link="robotiq_85_base_link" />
@@ -601,4 +667,15 @@
         <mimic joint="robotiq_85_left_knuckle_joint" multiplier="-1" />
     </joint>
+<!-- Add transmission for robotiq_85_right_knuckle_joint joint -->
+  <transmission name="robotiq_85_right_knuckle_joint_trans">
+    <type>transmission_interface/SimpleTransmission</type>
+    <joint name="robotiq_85_right_knuckle_joint">
+      <hardwareInterface>PositionJointInterface</hardwareInterface>
+    </joint>
+    <actuator name="robotiq_85_right_knuckle_joint_motor">
+      <hardwareInterface>PositionJointInterface</hardwareInterface>
+      <mechanicalReduction>1</mechanicalReduction>
+    </actuator>
+  </transmission>
     <joint name="robotiq_85_left_finger_joint" type="fixed">
         <parent link="robotiq_85_left_knuckle_link" />
@@ -639,3 +716,7 @@
         <mimic joint="robotiq_85_left_knuckle_joint" />
     </joint>
+	<!-- Gazebo plugin -->
+  <gazebo>
+    <plugin name="gazebo_ros_control" filename="libgazebo_ros_control.so"/>
+  </gazebo>
 </robot>

File: pharmacy_robot/urdf/pharmacy_robot.urdf.xacro (robot description, xacro)
@@ -72,5 +72,5 @@
         name="">
         <color
-          rgba="0.792156862745098 0.819607843137255 0.933333333333333 1" />
+          rgba="1 0 1 0.5" />
       </material>
     </visual>
@@ -93,4 +93,15 @@
   <dynamics damping="5" friction="3" />
 </joint>
+<!-- Add transmission for prismatic_base joint -->
+  <transmission name="prismatic_base_trans">
+    <type>transmission_interface/SimpleTransmission</type>
+    <joint name="prismatic_base">
+      <hardwareInterface>PositionJointInterface</hardwareInterface>
+    </joint>
+    <actuator name="prismatic_base_motor">
+      <hardwareInterface>PositionJointInterface</hardwareInterface>
+      <mechanicalReduction>1</mechanicalReduction>
+    </actuator>
+  </transmission>
   <link
     name="vertical_rail_link">
@@ -329,4 +340,15 @@
       <dynamics damping="5" friction="3" />
   </joint>
+  <!-- Add transmission for gripper_base joint -->
+  <transmission name="gripper_base_trans">
+    <type>transmission_interface/SimpleTransmission</type>
+    <joint name="gripper_base">
+      <hardwareInterface>PositionJointInterface</hardwareInterface>
+    </joint>
+    <actuator name="gripper_base_motor">
+      <hardwareInterface>PositionJointInterface</hardwareInterface>
+      <mechanicalReduction>1</mechanicalReduction>
+    </actuator>
+  </transmission>
   <link
     name="camera_link">
@@ -414,3 +436,7 @@
     </sensor>
   </gazebo>
+  <!-- Gazebo plugin -->
+  <gazebo>
+    <plugin name="gazebo_ros_control" filename="libgazebo_ros_control.so"/>
+  </gazebo>
 </robot>

Commit message: Added damping and friction to gripper joints

File: pharmacy_robot/urdf/pharmacy_gripper.xacro (robot description, xacro)
@@ -679,4 +679,5 @@
         <origin xyz="0.03060114 0.0 0.05490452" rpy="0 0 0" />
         <limit lower="0.0" upper="0.8" velocity="0.5" effort="50" />
+		<dynamics damping="5" friction="3" />
     </joint>
 	<!-- Add transmission for robotiq_85_left_knuckle_joint joint -->
@@ -698,4 +699,5 @@
         <limit lower="-0.8" upper="0.0" velocity="0.5" effort="50" />
         <mimic joint="robotiq_85_left_knuckle_joint" multiplier="-1" />
+		<dynamics damping="5" friction="3" />
     </joint>
 <!-- Add transmission for robotiq_85_right_knuckle_joint joint -->
@@ -726,4 +728,5 @@
         <origin xyz="0.0127 0.0 0.06142" rpy="0 0 0" />
         <mimic joint="robotiq_85_left_knuckle_joint" />
+		<dynamics damping="5" friction="3" />
     </joint>
     <joint name="robotiq_85_right_inner_knuckle_joint" type="continuous">
@@ -733,4 +736,5 @@
         <origin xyz="-0.0127 0.0 0.06142" rpy="0 0 0" />
         <mimic joint="robotiq_85_left_knuckle_joint" multiplier="-1" />
+		<dynamics damping="5" friction="3" />
     </joint>
     <joint name="robotiq_85_left_finger_tip_joint" type="continuous">
@@ -740,4 +744,5 @@
         <origin xyz="0.00563134 0.0 0.04718515" rpy="0 0 0" />
         <mimic joint="robotiq_85_left_knuckle_joint" multiplier="-1" />
+		<dynamics damping="5" friction="3" />
     </joint>
     <joint name="robotiq_85_right_finger_tip_joint" type="continuous">
@@ -747,4 +752,5 @@
         <origin xyz="-0.00563134 0.0 0.04718515" rpy="0 0 0" />
         <mimic joint="robotiq_85_left_knuckle_joint" />
+		<dynamics damping="5" friction="3" />
     </joint>
 	<!-- Gazebo plugin -->

Commit message: minor fixes

File: pharmacy_robot/urdf/pharmacy_gripper.xacro (robot description, xacro)
@@ -397,73 +397,73 @@
     </link>
     <link name="robotiq_85_left_finger_tip_link">
-        <visual>
-            <geometry>
-                <mesh filename="package://pharmacy_robot/meshes/gripper/visual/left_finger_tip.dae" />
-            </geometry>
-        </visual>
-        <collision>
-            <geometry>
-                <mesh filename="package://pharmacy_robot/meshes/gripper/collision/left_finger_tip.stl" />
-            </geometry>
-            <surface>
-                <friction>
+    <visual>
+        <geometry>
+            <mesh filename="package://pharmacy_robot/meshes/gripper/visual/left_finger_tip.dae" />
+        </geometry>
+    </visual>
+    <collision>
+        <geometry>
+            <mesh filename="package://pharmacy_robot/meshes/gripper/collision/left_finger_tip.stl" />
+        </geometry>
+        <surface>
+            <friction>
                 <ode>
-                    <mu1>100000.0</mu1>
-                    <mu2>100000.0</mu2>
+                    <mu>10</mu>
+                    <mu2>10</mu2>
                 </ode>
-                </friction>
-                <contact>
+            </friction>
+            <contact>
                 <ode>
-                    <kp>1e+5</kp>
-                    <kd>1</kd>
-                    <soft_cfm>0</soft_cfm>
-                    <soft_erp>0.2</soft_erp>
+                    <kp>50000</kp> <!-- Spring stiffness -->
+                    <kd>5</kd>    <!-- Damping -->
+                    <soft_cfm>0.00001</soft_cfm> <!-- Constraint Force Mixing -->
+                    <soft_erp>0.8</soft_erp>    <!-- Error Reduction Parameter -->
                     <minDepth>0.002</minDepth>
-                    <maxVel>0</maxVel>
+                    <maxVel>0.1</maxVel>
                 </ode>
-                </contact>
-            </surface>
-        </collision>
-        <inertial>
-            <origin xyz="-0.01456706 -0.0008 0.01649701" rpy="0 0 0" />
-            <mass value="4.268588744e-02" />
-            <inertia ixx="1.048152e-05" iyy="1.197888e-05" izz="4.22784e-06" ixy="0.0" ixz="3.5232e-6" iyz="0.0" />
-        </inertial>
-    </link>
-    <link name="robotiq_85_right_finger_tip_link">
-        <visual>
-            <geometry>
-                <mesh filename="package://pharmacy_robot/meshes/gripper/visual/right_finger_tip.dae" />
-            </geometry>
-        </visual>
-        <collision>
-            <geometry>
-                <mesh filename="package://pharmacy_robot/meshes/gripper/collision/right_finger_tip.stl" />
-            </geometry>
-            <surface>
-                <friction>
+            </contact>
+        </surface>
+    </collision>
+    <inertial>
+        <origin xyz="-0.01456706 -0.0008 0.01649701" rpy="0 0 0" />
+        <mass value="0.1" /> <!-- Increased for stability -->
+        <inertia ixx="1.2e-05" iyy="1.3e-05" izz="1.1e-05" ixy="0.0" ixz="3.5e-6" iyz="0.0" />
+    </inertial>
+</link>
+<link name="robotiq_85_right_finger_tip_link">
+    <visual>
+        <geometry>
+            <mesh filename="package://pharmacy_robot/meshes/gripper/visual/right_finger_tip.dae" />
+        </geometry>
+    </visual>
+    <collision>
+        <geometry>
+            <mesh filename="package://pharmacy_robot/meshes/gripper/collision/right_finger_tip.stl" />
+        </geometry>
+        <surface>
+            <friction>
                 <ode>
-                    <mu1>100000.0</mu1>
-                    <mu2>100000.0</mu2>
+                    <mu>10</mu>
+                    <mu2>10</mu2>
                 </ode>
-                </friction>
-                <contact>
+            </friction>
+            <contact>
                 <ode>
-                    <kp>1e+5</kp>
-                    <kd>1</kd>
-                    <soft_cfm>0</soft_cfm>
-                    <soft_erp>0.2</soft_erp>
+                    <kp>50000</kp>
+                    <kd>5</kd>
+                    <soft_cfm>0.00001</soft_cfm>
+                    <soft_erp>0.8</soft_erp>
                     <minDepth>0.002</minDepth>
-                    <maxVel>0</maxVel>
+                    <maxVel>0.1</maxVel>
                 </ode>
-                </contact>
-            </surface>
-        </collision>
-        <inertial>
-            <origin xyz="0.01456706 5e-05 0.01649701" rpy="0 0 0" />
-            <mass value="4.268588744e-02" />
-            <inertia ixx="1.048152e-05" iyy="1.197888e-05" izz="4.22784e-06" ixy="0.0" ixz="-3.5232e-06" iyz="0.0" />
-        </inertial>
-    </link>
+            </contact>
+        </surface>
+    </collision>
+    <inertial>
+        <origin xyz="0.01456706 5e-05 0.01649701" rpy="0 0 0" />
+        <mass value="0.1" />
+        <inertia ixx="1.2e-05" iyy="1.3e-05" izz="1.1e-05" ixy="0.0" ixz="-3.5e-6" iyz="0.0" />
+    </inertial>
+</link>
 	<!-- ********** JOINTS ********** -->
 	<joint name="robot_base" type="prismatic">
@@ -572,5 +572,5 @@
         <axis xyz="0 -1 0" />
         <origin xyz="0.03060114 0.0 0.05490452" rpy="0 0 0" />
-        <limit lower="0.0" upper="0.8" velocity="0.5" effort="50" />
+        <limit lower="0.0" upper="0.8" velocity="0.5" effort="5" />
 		<dynamics damping="5" friction="3" />
     </joint>
@@ -580,5 +580,5 @@
         <axis xyz="0 -1 0" />
         <origin xyz="-0.03060114 0.0 0.05490452" rpy="0 0 0" />
-        <limit lower="-0.8" upper="0.0" velocity="0.5" effort="50" />
+        <limit lower="-0.8" upper="0.0" velocity="0.5" effort="5" />
         <mimic joint="robotiq_85_left_knuckle_joint" multiplier="-1" />
 		<dynamics damping="5" friction="3" />
@@ -600,5 +600,5 @@
         <origin xyz="0.0127 0.0 0.06142" rpy="0 0 0" />
         <mimic joint="robotiq_85_left_knuckle_joint" />
-		<dynamics damping="5" friction="3" />
+		<dynamics damping="5" friction="1" />
     </joint>
     <joint name="robotiq_85_right_inner_knuckle_joint" type="continuous">
@@ -608,5 +608,5 @@
         <origin xyz="-0.0127 0.0 0.06142" rpy="0 0 0" />
         <mimic joint="robotiq_85_left_knuckle_joint" multiplier="-1" />
-		<dynamics damping="5" friction="3" />
+		<dynamics damping="5" friction="1" />
     </joint>
     <joint name="robotiq_85_left_finger_tip_joint" type="continuous">
@@ -616,5 +616,5 @@
         <origin xyz="0.00563134 0.0 0.04718515" rpy="0 0 0" />
         <mimic joint="robotiq_85_left_knuckle_joint" multiplier="-1" />
-		<dynamics damping="5" friction="3" />
+		<dynamics damping="5" friction="1" />
     </joint>
     <joint name="robotiq_85_right_finger_tip_joint" type="continuous">
@@ -624,5 +624,5 @@
         <origin xyz="-0.00563134 0.0 0.04718515" rpy="0 0 0" />
         <mimic joint="robotiq_85_left_knuckle_joint" />
-		<dynamics damping="5" friction="3" />
+		<dynamics damping="5" friction="1" />
     </joint>
 	<!--*********TRANSMISSIONS*************-->
